File: eagle-files/mainbd.sch (EAGLE design)
At the start: 24 parts, among them J1 4328, T1 3904, X1 TSW-102-07-G-S

Commit message: Statring work on adding IV-18 support
Parts:
- added R10, R8, R9: 10k, rcl:R-US_M0805
- added R11: 0, rcl:R-US_M0805
- added U$3: DS3231M, mgregg:DS3231M
- added U$5: BATTERY-2998-COIN, mgregg:BATTERY-2998-COIN
Connections:
- new net N$10: R9.2, U$3.INT
- new net N$14: R8.2, U$3.32KHZ
- new net N$9: R10.2, U$3.RST
- new net RTC-BAT: R11.1, U$3.VBAT, U$5.POS
- net 3V3: now also R10.1, R11.2, R8.1, R9.1, U$3.VCC
- net GND: now also U$3.GND, U$5.NEG
- net SCL: now also U$3.SCL
- net SDA: now also U$3.SDA
Changed lines of the file:
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@@
 <part name="U$9" library="mgregg" deviceset="DIODE-ZENIER-CMSH1-20MLTR13" device=""/>
 <part name="3.3V-LDO" library="mgregg" deviceset="LDO-3.3V-AZ1117CR-3.3TRG1" device=""/>
+<part name="U$3" library="mgregg" deviceset="DS3231M" device=""/>
+<part name="R8" library="rcl" library_urn="urn:adsk.eagle:library:334" deviceset="R-US_" device="M0805" package3d_urn="urn:adsk.eagle:package:23556/2" value="10k"/>
+<part name="R9" library="rcl" library_urn="urn:adsk.eagle:library:334" deviceset="R-US_" device="M0805" package3d_urn="urn:adsk.eagle:package:23556/2" value="10k"/>
+<part name="R10" library="rcl" library_urn="urn:adsk.eagle:library:334" deviceset="R-US_" device="M0805" package3d_urn="urn:adsk.eagle:package:23556/2" value="10k"/>
+<part name="U$5" library="mgregg" deviceset="BATTERY-2998-COIN" device=""/>
+<part name="R11" library="rcl" library_urn="urn:adsk.eagle:library:334" deviceset="R-US_" device="M0805" package3d_urn="urn:adsk.eagle:package:23556/2" value="0"/>
 </parts>
 <sheets>
@@
 <instance part="U$9" gate="G$1" x="182.88" y="-17.78" smashed="yes"/>
 <instance part="3.3V-LDO" gate="G$1" x="195.58" y="63.5" smashed="yes"/>
+<instance part="U$3" gate="G$1" x="111.76" y="-66.04" smashed="yes"/>
+<instance part="R8" gate="G$1" x="78.74" y="-60.96" smashed="yes">
+<attribute name="NAME" x="74.93" y="-59.4614" size="1.778" layer="95"/>
+<attribute name="VALUE" x="74.93" y="-64.262" size="1.778" layer="96"/>
+</instance>
+<instance part="R9" gate="G$1" x="78.74" y="-66.04" smashed="yes">
+<attribute name="NAME" x="74.93" y="-64.5414" size="1.778" layer="95"/>
+<attribute name="VALUE" x="74.93" y="-69.342" size="1.778" layer="96"/>
+</instance>
+<instance part="R10" gate="G$1" x="78.74" y="-68.58" smashed="yes">
+<attribute name="NAME" x="74.93" y="-67.0814" size="1.778" layer="95"/>
+<attribute name="VALUE" x="74.93" y="-71.882" size="1.778" layer="96"/>
+</instance>
+<instance part="U$5" gate="G$2" x="30.48" y="-60.96" smashed="yes"/>
+<instance part="R11" gate="G$1" x="53.34" y="-73.66" smashed="yes">
+<attribute name="NAME" x="49.53" y="-72.1614" size="1.778" layer="95"/>
+<attribute name="VALUE" x="49.53" y="-76.962" size="1.778" layer="96"/>
+</instance>
 </instances>
 <busses>
@@
 <wire x1="187.96" y1="63.5" x2="170.18" y2="63.5" width="0.1524" layer="91"/>
 <label x="172.72" y="63.5" size="1.778" layer="95"/>
+</segment>
+<segment>
+<pinref part="U$3" gate="G$1" pin="GND"/>
+<wire x1="101.6" y1="-78.74" x2="83.82" y2="-78.74" width="0.1524" layer="91"/>
+<label x="88.9" y="-78.74" size="1.778" layer="95"/>
+</segment>
+<segment>
+<pinref part="U$5" gate="G$2" pin="NEG"/>
+<wire x1="45.72" y1="-63.5" x2="60.96" y2="-63.5" width="0.1524" layer="91"/>
+<label x="50.8" y="-63.5" size="1.778" layer="95"/>
 </segment>
 </net>
@@
 <label x="172.72" y="66.04" size="1.778" layer="95"/>
 </segment>
+<segment>
+<pinref part="U$3" gate="G$1" pin="VCC"/>
+<wire x1="101.6" y1="-63.5" x2="83.82" y2="-63.5" width="0.1524" layer="91"/>
+<label x="88.9" y="-63.5" size="1.778" layer="95"/>
+</segment>
+<segment>
+<pinref part="R10" gate="G$1" pin="1"/>
+<pinref part="R9" gate="G$1" pin="1"/>
+<wire x1="73.66" y1="-68.58" x2="73.66" y2="-66.04" width="0.1524" layer="91"/>
+<pinref part="R8" gate="G$1" pin="1"/>
+<wire x1="73.66" y1="-66.04" x2="73.66" y2="-60.96" width="0.1524" layer="91"/>
+<junction x="73.66" y="-66.04"/>
+<wire x1="73.66" y1="-60.96" x2="68.58" y2="-60.96" width="0.1524" layer="91"/>
+<junction x="73.66" y="-60.96"/>
+<label x="68.58" y="-60.96" size="1.778" layer="95"/>
+</segment>
+<segment>
+<pinref part="R11" gate="G$1" pin="2"/>
+<wire x1="58.42" y1="-73.66" x2="66.04" y2="-73.66" width="0.1524" layer="91"/>
+<label x="60.96" y="-73.66" size="1.778" layer="95"/>
+</segment>
 </net>
 <net name="SCL" class="0">
@@
 <label x="2.54" y="5.08" size="1.778" layer="95"/>
 </segment>
+<segment>
+<pinref part="U$3" gate="G$1" pin="SCL"/>
+<wire x1="101.6" y1="-71.12" x2="83.82" y2="-71.12" width="0.1524" layer="91"/>
+<label x="88.9" y="-71.12" size="1.778" layer="95"/>
+</segment>
 </net>
 <net name="SDA" class="0">
@@
 <wire x1="12.7" y1="7.62" x2="0" y2="7.62" width="0.1524" layer="91"/>
 <label x="2.54" y="7.62" size="1.778" layer="95"/>
+</segment>
+<segment>
+<pinref part="U$3" gate="G$1" pin="SDA"/>
+<wire x1="101.6" y1="-73.66" x2="83.82" y2="-73.66" width="0.1524" layer="91"/>
+<label x="88.9" y="-73.66" size="1.778" layer="95"/>
 </segment>
 </net>
@@
 </segment>
 </net>
+<net name="RTC-BAT" class="0">
+<segment>
+<pinref part="U$3" gate="G$1" pin="VBAT"/>
+<wire x1="101.6" y1="-76.2" x2="83.82" y2="-76.2" width="0.1524" layer="91"/>
+<label x="88.9" y="-76.2" size="1.778" layer="95"/>
+</segment>
+<segment>
+<pinref part="U$5" gate="G$2" pin="POS"/>
+<wire x1="45.72" y1="-58.42" x2="60.96" y2="-58.42" width="0.1524" layer="91"/>
+<label x="50.8" y="-58.42" size="1.778" layer="95"/>
+</segment>
+<segment>
+<pinref part="R11" gate="G$1" pin="1"/>
+<wire x1="48.26" y1="-73.66" x2="38.1" y2="-73.66" width="0.1524" layer="91"/>
+<label x="40.64" y="-73.66" size="1.778" layer="95"/>
+</segment>
+</net>
+<net name="N$9" class="0">
+<segment>
+<pinref part="U$3" gate="G$1" pin="RST"/>
+<wire x1="101.6" y1="-68.58" x2="83.82" y2="-68.58" width="0.1524" layer="91"/>
+<label x="88.9" y="-68.58" size="1.778" layer="95"/>
+<pinref part="R10" gate="G$1" pin="2"/>
+<junction x="83.82" y="-68.58"/>
+</segment>
+</net>
+<net name="N$10" class="0">
+<segment>
+<pinref part="U$3" gate="G$1" pin="INT"/>
+<wire x1="101.6" y1="-66.04" x2="83.82" y2="-66.04" width="0.1524" layer="91"/>
+<label x="88.9" y="-66.04" size="1.778" layer="95"/>
+<pinref part="R9" gate="G$1" pin="2"/>
+<junction x="83.82" y="-66.04"/>
+</segment>
+</net>
+<net name="N$14" class="0">
+<segment>
+<pinref part="U$3" gate="G$1" pin="32KHZ"/>
+<wire x1="101.6" y1="-60.96" x2="83.82" y2="-60.96" width="0.1524" layer="91"/>
+<label x="88.9" y="-60.96" size="1.778" layer="95"/>
+<pinref part="R8" gate="G$1" pin="2"/>
+</segment>
+</net>
