File: eagle-files/iv-18.brd (EAGLE design)
At the start: 28 x 40 mm, 2 parts

Commit message: Adding cam file for production
Routing:
- net G3: track 0.00 -> 40.9 mm
- net B: track 0.00 -> 40.0 mm
- net G: track 0.00 -> 39.8 mm
- net F1: track 0.00 -> 39.0 mm
- net G9: track 0.00 -> 37.8 mm
- net G1: track 0.00 -> 36.1 mm
- net D: track 0.00 -> 36.1 mm
- net C: track 0.00 -> 35.0 mm, vias 0 -> 2
- net DP: track 0.00 -> 33.8 mm, vias 0 -> 4
- net A: track 0.00 -> 29.5 mm, vias 0 -> 1
- net G5: track 0.00 -> 28.2 mm, vias 0 -> 1
- net G8: track 0.00 -> 27.6 mm, vias 0 -> 1
- net G2: track 0.00 -> 25.1 mm, vias 0 -> 1
- net G6: track 0.00 -> 24.6 mm
- net G7: track 0.00 -> 23.7 mm, vias 0 -> 1
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- added copper zone on layer 1, net GND
- added copper zone on layer 16, net GND
Other:
- board size 28 x 40 mm -> 28 x 40.1 mm
- board text added: "A"
- board text added: "B"
- board text added: "IV-18"
